File: UccMicroDuino/UccMicroDuino.kicad_pcb (KiCad board)
At the start: 2 copper layers, 45 x 45.2 mm, 14 parts, among them J1 USB_PCB_A, J2 Header, U1 ATtiny85-20S

Commit message: PCB finalizado
Parts:
- moved R2 36.6 mm to (126.0, 67.5), turned to 90 degrees
- moved C1 35.6 mm to (133.0, 95.0)
- moved D1 35.2 mm to (128.5, 96.0), turned to -90 degrees
- moved D2 35.0 mm to (130.5, 67.5), turned to 90 degrees
- moved R5 33.8 mm to (138.5, 92.0), turned to 180 degrees
- moved J1 32.5 mm to (117.2, 97.5)
- moved J2 31.7 mm to (152.5, 95.7), turned to 180 degrees
- moved D5 30.8 mm to (135.5, 101.0), turned to -90 degrees
- moved R4 27.6 mm to (144.0, 97.5), turned to -90 degrees
- moved D3 27.5 mm to (126.5, 101.5)
- moved D4 24.1 mm to (145.0, 85.5), turned to 90 degrees
- moved R3 22.0 mm to (128.0, 82.5), turned to 180 degrees
- moved R1 21.3 mm to (128.0, 77.0)
- moved U1 12.5 mm to (143.0, 69.5), turned to -90 degrees
Routing:
- net GND: track 2.58 -> 133.4 mm
- net +5V: track 0.00 -> 73.6 mm
- net Net-(J2-Pin_8): track 0.00 -> 42.1 mm
- net Net-(D2-K): track 0.35 -> 38.1 mm
- net Net-(J2-Pin_7): track 0.00 -> 36.5 mm
- net Net-(D1-K): track 0.00 -> 31.4 mm
- net Net-(J2-Pin_4): track 0.00 -> 23.5 mm
- net Net-(D4-A): track 0.00 -> 20.4 mm
- net Net-(J2-Pin_6): track 0.00 -> 16.2 mm
- net Net-(J2-Pin_9): track 0.00 -> 12.6 mm
- net Net-(D5-K): track 0.00 -> 8.79 mm
- net Net-(D3-A): track 0.00 -> 7.96 mm
- net Net-(D4-K): track 0.00 -> 7.45 mm
Other:
- board size 45 x 45.2 mm -> 45 x 45 mm
